Commit message: Add ros2_control and Robotiq gripper integration
- Added ros2_control with fake hardware for 6 arm joints + gripper
- Added JointTrajectoryController for arm
- Added GripperActionController for gripper
- Added Robotiq 2F-85 gripper links attached to tool0
- Updated bringup.launch.py with all controller spawners

File: src/fanuc_crx10ia_description/urdf/crx10ial.urdf (robot description, URDF)
Before this commit: robot fanuc_crx10ial, 10 links, 9 joints
Links:
- added link gripper_base_link; collision box size=0.04 0.09 0.04; visual box size=0.04 0.09 0.04
- added link gripper_left_finger_link; collision box size=0.02 0.02 0.08; visual box size=0.02 0.02 0.08
- added link gripper_right_finger_link; collision box size=0.02 0.02 0.08; visual box size=0.02 0.02 0.08
Joints:
- added joint gripper_base_joint: type fixed, parent tool0, child gripper_base_link, origin xyz=0 0 0 rpy=0 0 0
- added joint gripper_finger_joint: type prismatic, parent gripper_base_link, child gripper_left_finger_link, origin xyz=0 0.0425 0.04 rpy=0 0 0, axis 0 -1 0, limit lower=0.0 upper=0.04 effort=100 velocity=0.1
- added joint gripper_right_finger_joint: type prismatic, parent gripper_base_link, child gripper_right_finger_link, origin xyz=0 -0.0425 0.04 rpy=0 0 0, axis 0 1 0, limit lower=0.0 upper=0.04 effort=100 velocity=0.1, mimic joint=gripper_finger_joint multiplier=1 offset=0
