Commit message: initial run

File: src/fanuc_dual_arm_description/urdf/crx10ia_macro.xacro (robot description, xacro)
@@ -20,4 +20,13 @@
         </geometry>
       </collision>
+      <visual>
+        <origin rpy="0 0 0" xyz="0 0 0.355"/>
+        <geometry>
+          <cylinder radius="0.05" length="0.41"/>
+        </geometry>
+        <material name="${prefix}white">
+          <color rgba="0.86 0.85 0.81 1.0"/>
+        </material>
+      </visual>
     </link>
     <joint name="${prefix}base_joint" type="fixed">
@@ -108,5 +117,5 @@
     <!-- Arm joints -->
     <joint name="${prefix}joint_1" type="revolute">
-      <origin rpy="0 0 0" xyz="0 0 0.245"/>
+      <origin rpy="0 0 0" xyz="0 0 0.710"/>
       <parent link="${prefix}base_link"/>
       <child link="${prefix}link_1"/>

File: src/fanuc_dual_arm_description/urdf/dual_arm.urdf.xacro (robot description, xacro)
@@ -22,12 +22,29 @@
     <child link="platform"/>
   </joint>
-  <!-- Left arm (Robot B): tilted 45° towards the LEFT side (outward) -->
+  <!-- Left arm (Robot B): tilted 45° outward (ROLL around X-axis) -->
   <xacro:crx10ia_arm prefix="left_" parent_link="platform">
-    <origin xyz="-0.4 0 0" rpy="0 -0.785 0"/>
+    <origin xyz="0 -0.15 0" rpy="0.785 0 0"/>
   </xacro:crx10ia_arm>
-  <!-- Right arm (Robot A): tilted 45° towards the RIGHT side (outward, mirror image) -->
+  <!-- Right arm (Robot A): tilted 45° outward (ROLL around X-axis, mirror) -->
   <xacro:crx10ia_arm prefix="right_" parent_link="platform">
-    <origin xyz="0.4 0 0" rpy="0 0.785 0"/>
+    <origin xyz="0 0.15 0" rpy="-0.785 0 0"/>
   </xacro:crx10ia_arm>
+  <!-- Workpiece: A stick/cylinder for pick-and-place demo -->
+  <link name="workpiece">
+    <visual>
+      <origin rpy="0 1.57 0" xyz="0 0 0"/>
+      <geometry>
+        <cylinder radius="0.02" length="0.3"/>
+      </geometry>
+      <material name="workpiece_blue">
+        <color rgba="0.2 0.4 0.8 1.0"/>
+      </material>
+    </visual>
+  </link>
+  <joint name="workpiece_joint" type="fixed">
+    <origin rpy="0 0 0" xyz="0.5 0 0.15"/>
+    <parent link="world"/>
+    <child link="workpiece"/>
+  </joint>
   <!-- ros2_control for both arms -->
   <ros2_control name="DualArmSystem" type="system">
@@ -38,10 +55,10 @@
     <joint name="left_joint_1">
       <command_interface name="position"/>
-      <state_interface name="position"><param name="initial_value">0.0</param></state_interface>
+      <state_interface name="position"><param name="initial_value">-0.017</param></state_interface>
       <state_interface name="velocity"/>
     </joint>
     <joint name="left_joint_2">
       <command_interface name="position"/>
-      <state_interface name="position"><param name="initial_value">0.0</param></state_interface>
+      <state_interface name="position"><param name="initial_value">1.614</param></state_interface>
       <state_interface name="velocity"/>
     </joint>
@@ -53,5 +70,5 @@
     <joint name="left_joint_4">
       <command_interface name="position"/>
-      <state_interface name="position"><param name="initial_value">0.0</param></state_interface>
+      <state_interface name="position"><param name="initial_value">-3.209</param></state_interface>
       <state_interface name="velocity"/>
     </joint>
@@ -74,25 +91,25 @@
     <joint name="right_joint_1">
       <command_interface name="position"/>
-      <state_interface name="position"><param name="initial_value">0.0</param></state_interface>
+      <state_interface name="position"><param name="initial_value">-3.142</param></state_interface>
       <state_interface name="velocity"/>
     </joint>
     <joint name="right_joint_2">
       <command_interface name="position"/>
-      <state_interface name="position"><param name="initial_value">0.0</param></state_interface>
+      <state_interface name="position"><param name="initial_value">-1.580</param></state_interface>
       <state_interface name="velocity"/>
     </joint>
     <joint name="right_joint_3">
       <command_interface name="position"/>
-      <state_interface name="position"><param name="initial_value">0.0</param></state_interface>
+      <state_interface name="position"><param name="initial_value">-3.031</param></state_interface>
       <state_interface name="velocity"/>
     </joint>
     <joint name="right_joint_4">
       <command_interface name="position"/>
-      <state_interface name="position"><param name="initial_value">0.0</param></state_interface>
+      <state_interface name="position"><param name="initial_value">-3.029</param></state_interface>
       <state_interface name="velocity"/>
     </joint>
     <joint name="right_joint_5">
       <command_interface name="position"/>
-      <state_interface name="position"><param name="initial_value">0.0</param></state_interface>
+      <state_interface name="position"><param name="initial_value">0.085</param></state_interface>
       <state_interface name="velocity"/>
     </joint>

Commit message: both tasks donegit add . and mainly solved object collision issues with arms and gripper

File: src/fanuc_dual_arm_description/urdf/crx10ia_macro.xacro (robot description, xacro)
@@ -200,25 +200,25 @@
     </link>
     <joint name="${prefix}gripper_finger_joint" type="prismatic">
-      <origin rpy="0 0 0" xyz="0 0.0425 0.04"/>
+      <origin rpy="0 0 0" xyz="0 0.01 0.04"/>
       <parent link="${prefix}gripper_base_link"/>
       <child link="${prefix}gripper_left_finger_link"/>
+      <axis xyz="0 1 0"/>
+      <limit effort="100" lower="0.0" upper="0.04" velocity="0.1"/>
+    </joint>
+    <link name="${prefix}gripper_right_finger_link">
+      <visual>
+        <origin rpy="0 0 0" xyz="0 0 0.04"/>
+        <geometry>
+          <box size="0.02 0.02 0.08"/>
+        </geometry>
+        <material name="${prefix}finger_grey"/>
+      </visual>
+    </link>
+    <joint name="${prefix}gripper_right_finger_joint" type="prismatic">
+      <origin rpy="0 0 0" xyz="0 -0.01 0.04"/>
+      <parent link="${prefix}gripper_base_link"/>
+      <child link="${prefix}gripper_right_finger_link"/>
       <axis xyz="0 -1 0"/>
       <limit effort="100" lower="0.0" upper="0.04" velocity="0.1"/>
-    </joint>
-    <link name="${prefix}gripper_right_finger_link">
-      <visual>
-        <origin rpy="0 0 0" xyz="0 0 0.04"/>
-        <geometry>
-          <box size="0.02 0.02 0.08"/>
-        </geometry>
-        <material name="${prefix}finger_grey"/>
-      </visual>
-    </link>
-    <joint name="${prefix}gripper_right_finger_joint" type="prismatic">
-      <origin rpy="0 0 0" xyz="0 -0.0425 0.04"/>
-      <parent link="${prefix}gripper_base_link"/>
-      <child link="${prefix}gripper_right_finger_link"/>
-      <axis xyz="0 1 0"/>
-      <limit effort="100" lower="0.0" upper="0.04" velocity="0.1"/>
       <mimic joint="${prefix}gripper_finger_joint" multiplier="1" offset="0"/>
     </joint>
